Commit message: for building mesh

File: masterHumanoid2025_description/urdf/masterHumanoid2025.xacro (robot description, xacro)
@@ -6,7 +6,7 @@
 <link name="base_link">
   <inertial>
-    <origin xyz="-0.0019277625580420743 -0.0002828648876733997 0.690502612360238" rpy="0 0 0"/>
+    <origin xyz="0.012834207217545641 -0.00028286488702963016 0.6512228716334499" rpy="0 0 0"/>
     <mass value="5.614608211157563"/>
-    <inertia ixx="0.296093" iyy="0.167039" izz="0.152631" ixy="0.000112" iyz="-0.000108" ixz="0.001772"/>
+    <inertia ixx="0.295311" iyy="0.167039" izz="0.153413" ixy="0.000102" iyz="-0.000117" ixz="-0.010711"/>
   </inertial>
   <visual>
@@ -26,10 +26,10 @@
 <link name="left_upper_frame_1">
   <inertial>
-    <origin xyz="-0.005046700831779199 1.0557817920323065e-05 -0.02143088061471432" rpy="0 0 0"/>
-    <mass value="0.1555228615666778"/>
-    <inertia ixx="0.000129" iyy="0.000495" izz="0.000449" ixy="0.0" iyz="0.0" ixz="-3e-05"/>
-  </inertial>
-  <visual>
-    <origin xyz="0.009035 -0.07965 -0.648137" rpy="0 0 0"/>
+    <origin xyz="-0.00689471238167166 1.055781750963769e-05 -0.02090957090882195" rpy="0 0 0"/>
+    <mass value="0.15552286156667774"/>
+    <inertia ixx="0.000126" iyy="0.000495" izz="0.000452" ixy="0.0" iyz="-0.0" ixz="-2e-06"/>
+  </inertial>
+  <visual>
+    <origin xyz="-0.002061 -0.07965 -0.609638" rpy="0 0 0"/>
     <geometry>
       <mesh filename="file://$(find masterHumanoid2025_description)/meshes/left_upper_frame_1.stl" scale="0.001 0.001 0.001"/>
@@ -38,5 +38,5 @@
   </visual>
   <collision>
-    <origin xyz="0.009035 -0.07965 -0.648137" rpy="0 0 0"/>
+    <origin xyz="-0.002061 -0.07965 -0.609638" rpy="0 0 0"/>
     <geometry>
       <mesh filename="file://$(find masterHumanoid2025_description)/meshes/left_upper_frame_1.stl" scale="0.001 0.001 0.001"/>
@@ -46,10 +46,10 @@
 <link name="right_upper_frame_1">
   <inertial>
-    <origin xyz="-0.0050467103826035645 3.918892784643413e-06 -0.021430880698611654" rpy="0 0 0"/>
+    <origin xyz="-0.0068947219033479515 3.918892374304983e-06 -0.020909570157323865" rpy="0 0 0"/>
     <mass value="0.1555228610526311"/>
-    <inertia ixx="0.000129" iyy="0.000495" izz="0.000449" ixy="1e-06" iyz="0.0" ixz="-3e-05"/>
-  </inertial>
-  <visual>
-    <origin xyz="0.009035 0.08035 -0.648137" rpy="0 0 0"/>
+    <inertia ixx="0.000126" iyy="0.000495" izz="0.000452" ixy="1e-06" iyz="0.0" ixz="-2e-06"/>
+  </inertial>
+  <visual>
+    <origin xyz="-0.002061 0.08035 -0.609638" rpy="0 0 0"/>
     <geometry>
       <mesh filename="file://$(find masterHumanoid2025_description)/meshes/right_upper_frame_1.stl" scale="0.001 0.001 0.001"/>
@@ -58,5 +58,5 @@
   </visual>
   <collision>
-    <origin xyz="0.009035 0.08035 -0.648137" rpy="0 0 0"/>
+    <origin xyz="-0.002061 0.08035 -0.609638" rpy="0 0 0"/>
     <geometry>
       <mesh filename="file://$(find masterHumanoid2025_description)/meshes/right_upper_frame_1.stl" scale="0.001 0.001 0.001"/>
@@ -66,10 +66,10 @@
 <link name="left_upper_gearbox_1">
   <inertial>
-    <origin xyz="0.05679763300573742 0.0010494997385310512 -0.02259314565567294" rpy="0 0 0"/>
-    <mass value="0.7539590478154932"/>
-    <inertia ixx="0.000908" iyy="0.00133" izz="0.001405" ixy="3.5e-05" iyz="2.1e-05" ixz="-6.9e-05"/>
-  </inertial>
-  <visual>
-    <origin xyz="0.070085 -0.079715 -0.583137" rpy="0 0 0"/>
+    <origin xyz="0.05461317742426483 0.0010494997370183168 -0.02745729931198171" rpy="0 0 0"/>
+    <mass value="0.7539590478154929"/>
+    <inertia ixx="0.0009" iyy="0.00133" izz="0.001413" ixy="3.6e-05" iyz="1.8e-05" ixz="-2.5e-05"/>
+  </inertial>
+  <visual>
+    <origin xyz="0.064422 -0.079715 -0.550206" rpy="0 0 0"/>
     <geometry>
       <mesh filename="file://$(find masterHumanoid2025_description)/meshes/left_upper_gearbox_1.stl" scale="0.001 0.001 0.001"/>
@@ -78,5 +78,5 @@
   </visual>
   <collision>
-    <origin xyz="0.070085 -0.079715 -0.583137" rpy="0 0 0"/>
+    <origin xyz="0.064422 -0.079715 -0.550206" rpy="0 0 0"/>
     <geometry>
       <mesh filename="file://$(find masterHumanoid2025_description)/meshes/left_upper_gearbox_1.stl" scale="0.001 0.001 0.001"/>
@@ -86,10 +86,10 @@
 <link name="right_upper_gearbox_1">
   <inertial>
-    <origin xyz="0.057294496913915735 -0.0012029091034558848 -0.022593661068604054" rpy="0 0 0"/>
-    <mass value="0.7539598848625294"/>
-    <inertia ixx="0.000908" iyy="0.00133" izz="0.001405" ixy="-3.3e-05" iyz="-2.1e-05" ixz="-6.9e-05"/>
-  </inertial>
-  <visual>
-    <origin xyz="0.070085 0.080239 -0.583137" rpy="0 0 0"/>
+    <origin xyz="0.05510810569418474 -0.001202909104967953 -0.027501117303870726" rpy="0 0 0"/>
+    <mass value="0.7539598848625293"/>
+    <inertia ixx="0.0009" iyy="0.00133" izz="0.001413" ixy="-3.5e-05" iyz="-1.8e-05" ixz="-2.5e-05"/>
+  </inertial>
+  <visual>
+    <origin xyz="0.064422 0.080239 -0.550206" rpy="0 0 0"/>
     <geometry>
       <mesh filename="file://$(find masterHumanoid2025_description)/meshes/right_upper_gearbox_1.stl" scale="0.001 0.001 0.001"/>
@@ -98,5 +98,5 @@
   </visual>
   <collision>
-    <origin xyz="0.070085 0.080239 -0.583137" rpy="0 0 0"/>
+    <origin xyz="0.064422 0.080239 -0.550206" rpy="0 0 0"/>
     <geometry>
       <mesh filename="file://$(find masterHumanoid2025_description)/meshes/right_upper_gearbox_1.stl" scale="0.001 0.001 0.001"/>
@@ -106,10 +106,10 @@
 <link name="right_middle_leg_1">
   <inertial>
-    <origin xyz="0.0129261417013413 0.0503956601070247 -0.17114233911271742" rpy="0 0 0"/>
+    <origin xyz="-0.002039057333556183 0.05039566010299555 -0.1716171695275195" rpy="0 0 0"/>
     <mass value="1.077312188551498"/>
-    <inertia ixx="0.005505" iyy="0.004327" izz="0.001628" ixy="-2e-06" iyz="-2e-06" ixz="0.000186"/>
-  </inertial>
-  <visual>
-    <origin xyz="-0.02074 0.130854 -0.582791" rpy="0 0 0"/>
+    <inertia ixx="0.005508" iyy="0.004327" izz="0.001626" ixy="-2e-06" iyz="-1e-06" ixz="-0.000154"/>
+  </inertial>
+  <visual>
+    <origin xyz="-0.026028 0.130854 -0.541945" rpy="0 0 0"/>
     <geometry>
       <mesh filename="file://$(find masterHumanoid2025_description)/meshes/right_middle_leg_1.stl" scale="0.001 0.001 0.001"/>
@@ -118,5 +118,5 @@
   </visual>
   <collision>
-    <origin xyz="-0.02074 0.130854 -0.582791" rpy="0 0 0"/>
+    <origin xyz="-0.026028 0.130854 -0.541945" rpy="0 0 0"/>
     <geometry>
       <mesh filename="file://$(find masterHumanoid2025_description)/meshes/right_middle_leg_1.stl" scale="0.001 0.001 0.001"/>
@@ -126,10 +126,10 @@
 <link name="left_middle_leg_1">
   <inertial>
-    <origin xyz="0.013291361449427885 -0.05034809076935265 -0.17112828814454834" rpy="0 0 0"/>
-    <mass value="1.077312207009041"/>
-    <inertia ixx="0.005504" iyy="0.004327" izz="0.00163" ixy="-1e-06" iyz="2e-06" ixz="0.000197"/>
-  </inertial>
-  <visual>
-    <origin xyz="-0.020385 -0.130069 -0.582816" rpy="0 0 0"/>
+    <origin xyz="-0.0016744729586776093 -0.050348090773382356 -0.1716351578724804" rpy="0 0 0"/>
+    <mass value="1.077312207009042"/>
+    <inertia ixx="0.005509" iyy="0.004327" izz="0.001625" ixy="-1e-06" iyz="3e-06" ixz="-0.000142"/>
+  </inertial>
+  <visual>
+    <origin xyz="-0.025677 -0.130069 -0.542001" rpy="0 0 0"/>
     <geometry>
       <mesh filename="file://$(find masterHumanoid2025_description)/meshes/left_middle_leg_1.stl" scale="0.001 0.001 0.001"/>
@@ -138,5 +138,5 @@
   </visual>
   <collision>
-    <origin xyz="-0.020385 -0.130069 -0.582816" rpy="0 0 0"/>
+    <origin xyz="-0.025677 -0.130069 -0.542001" rpy="0 0 0"/>
     <geometry>
       <mesh filename="file://$(find masterHumanoid2025_description)/meshes/left_middle_leg_1.stl" scale="0.001 0.001 0.001"/>
@@ -146,10 +146,10 @@
 <link name="left_lower_leg_1">
   <inertial>
-    <origin xyz="-0.005976086031339919 -0.050405366889918674 -0.08985471728805111" rpy="0 0 0"/>
-    <mass value="0.5227872807967037"/>
-    <inertia ixx="0.001799" iyy="0.001164" izz="0.000784" ixy="-1e-06" iyz="0.0" ixz="4.2e-05"/>
-  </inertial>
-  <visual>
-    <origin xyz="-0.020101 -0.130312 -0.332816" rpy="0 0 0"/>
+    <origin xyz="-0.013784998532198027 -0.050405366896745935 -0.08899251108621237" rpy="0 0 0"/>
+    <mass value="0.5227872807967039"/>
+    <inertia ixx="0.001799" iyy="0.001164" izz="0.000785" ixy="-1e-06" iyz="0.0" ixz="-4.7e-05"/>
+  </inertial>
+  <visual>
+    <origin xyz="-0.003605 -0.130312 -0.292978" rpy="0 0 0"/>
     <geometry>
       <mesh filename="file://$(find masterHumanoid2025_description)/meshes/left_lower_leg_1.stl" scale="0.001 0.001 0.001"/>
@@ -158,5 +158,5 @@
   </visual>
   <collision>
-    <origin xyz="-0.020101 -0.130312 -0.332816" rpy="0 0 0"/>
+    <origin xyz="-0.003605 -0.130312 -0.292978" rpy="0 0 0"/>
     <geometry>
       <mesh filename="file://$(find masterHumanoid2025_description)/meshes/left_lower_leg_1.stl" scale="0.001 0.001 0.001"/>
@@ -166,10 +166,10 @@
 <link name="right_lower_leg_1">
   <inertial>
-    <origin xyz="-0.005830783148732369 0.050467821012633265 -0.08982985681998587" rpy="0 0 0"/>
+    <origin xyz="-0.013637598547290068 0.0504678210058071 -0.08897924378035954" rpy="0 0 0"/>
     <mass value="0.5227872807963939"/>
-    <inertia ixx="0.001799" iyy="0.001164" izz="0.000784" ixy="-1e-06" iyz="-0.0" ixz="4.2e-05"/>
-  </inertial>
-  <visual>
-    <origin xyz="-0.01971 0.130971 -0.332793" rpy="0 0 0"/>
+    <inertia ixx="0.001799" iyy="0.001164" izz="0.000785" ixy="-1e-06" iyz="-0.0" ixz="-4.7e-05"/>
+  </inertial>
+  <visual>
+    <origin xyz="-0.003213 0.130971 -0.292988" rpy="0 0 0"/>
     <geometry>
       <mesh filename="file://$(find masterHumanoid2025_description)/meshes/right_lower_leg_1.stl" scale="0.001 0.001 0.001"/>
@@ -178,5 +178,5 @@
   </visual>
   <collision>
-    <origin xyz="-0.01971 0.130971 -0.332793" rpy="0 0 0"/>
+    <origin xyz="-0.003213 0.130971 -0.292988" rpy="0 0 0"/>
     <geometry>
       <mesh filename="file://$(find masterHumanoid2025_description)/meshes/right_lower_leg_1.stl" scale="0.001 0.001 0.001"/>
@@ -184,12 +184,32 @@
   </collision>
 </link>
+<link name="right_lower_gearbox_1">
+  <inertial>
+    <origin xyz="-0.031464146139689994 0.051709582806054394 0.025036773942110124" rpy="0 0 0"/>
+    <mass value="0.7539594536633326"/>
+    <inertia ixx="0.000924" iyy="0.00133" izz="0.001389" ixy="3.3e-05" iyz="-2.4e-05" ixz="0.000111"/>
+  </inertial>
+  <visual>
+    <origin xyz="0.018569 0.131089 -0.044016" rpy="0 0 0"/>
+    <geometry>
+      <mesh filename="file://$(find masterHumanoid2025_description)/meshes/right_lower_gearbox_1.stl" scale="0.001 0.001 0.001"/>
+    </geometry>
+    <material name="silver"/>
+  </visual>
+  <collision>
+    <origin xyz="0.018569 0.131089 -0.044016" rpy="0 0 0"/>
+    <geometry>
+      <mesh filename="file://$(find masterHumanoid2025_description)/meshes/right_lower_gearbox_1.stl" scale="0.001 0.001 0.001"/>
+    </geometry>
+  </collision>
+</link>
 <link name="left_lower_gearbox_1">
   <inertial>
-    <origin xyz="-0.033526419385759954 0.05170958281515828 0.022199596774821334" rpy="0 0 0"/>
-    <mass value="0.753959453663333"/>
-    <inertia ixx="0.000908" iyy="0.00133" izz="0.001405" ixy="3.5e-05" iyz="-2.1e-05" ixz="6.9e-05"/>
-  </inertial>
-  <visual>
-    <origin xyz="-0.01971 0.131089 -0.082869" rpy="0 0 0"/>
+    <origin xyz="-0.03161463163781425 -0.05162366210071047 0.02502425476994688" rpy="0 0 0"/>
+    <mass value="0.7539594232725968"/>
+    <inertia ixx="0.000924" iyy="0.00133" izz="0.001389" ixy="-3.2e-05" iyz="2.4e-05" ixz="0.000111"/>
+  </inertial>
+  <visual>
+    <origin xyz="0.018177 -0.130555 -0.044005" rpy="0 0 0"/>
     <geometry>
       <mesh filename="file://$(find masterHumanoid2025_description)/meshes/left_lower_gearbox_1.stl" scale="0.001 0.001 0.001"/>
@@ -198,5 +218,5 @@
   </visual>
   <collision>
-    <origin xyz="-0.01971 0.131089 -0.082869" rpy="0 0 0"/>
+    <origin xyz="0.018177 -0.130555 -0.044005" rpy="0 0 0"/>
     <geometry>
       <mesh filename="file://$(find masterHumanoid2025_description)/meshes/left_lower_gearbox_1.stl" scale="0.001 0.001 0.001"/>
@@ -204,21 +224,21 @@
   </collision>
 </link>
-<link name="right_lower_gearbox_1">
-  <inertial>
-    <origin xyz="-0.03367477408867826 -0.05162366209160814 0.022174216478641956" rpy="0 0 0"/>
-    <mass value="0.7539594232725966"/>
-    <inertia ixx="0.000908" iyy="0.00133" izz="0.001405" ixy="-3.4e-05" iyz="2.1e-05" ixz="6.9e-05"/>
-  </inertial>
-  <visual>
-    <origin xyz="-0.020101 -0.130555 -0.082892" rpy="0 0 0"/>
-    <geometry>
-      <mesh filename="file://$(find masterHumanoid2025_description)/meshes/right_lower_gearbox_1.stl" scale="0.001 0.001 0.001"/>
-    </geometry>
-    <material name="silver"/>
-  </visual>
-  <collision>
-    <origin xyz="-0.020101 -0.130555 -0.082892" rpy="0 0 0"/>
-    <geometry>
-      <mesh filename="file://$(find masterHumanoid2025_description)/meshes/right_lower_gearbox_1.stl" scale="0.001 0.001 0.001"/>
+<link name="right_foot_1">
+  <inertial>
+    <origin xyz="0.06322056024770292 -0.00948657106036395 -0.06587835514287177" rpy="0 0 0"/>
+    <mass value="1.3311575432838632"/>
+    <inertia ixx="0.002293" iyy="0.007731" izz="0.008918" ixy="5.1e-05" iyz="-9.3e-05" ixz="0.000807"/>
+  </inertial>
+  <visual>
+    <origin xyz="0.109581 0.080373 -0.051583" rpy="0 0 0"/>
+    <geometry>
+      <mesh filename="file://$(find masterHumanoid2025_description)/meshes/right_foot_1.stl" scale="0.001 0.001 0.001"/>
+    </geometry>
+    <material name="silver"/>
+  </visual>
+  <collision>
+    <origin xyz="0.109581 0.080373 -0.051583" rpy="0 0 0"/>
+    <geometry>
+      <mesh filename="file://$(find masterHumanoid2025_description)/meshes/right_foot_1.stl" scale="0.001 0.001 0.001"/>
     </geometry>
   </collision>
@@ -226,10 +246,10 @@
 <link name="left_foot_1">
   <inertial>
-    <origin xyz="0.06872157934204118 -0.009486571049873826 -0.06011727006259174" rpy="0 0 0"/>
-    <mass value="1.3311575432838623"/>
-    <inertia ixx="0.002203" iyy="0.007731" izz="0.009008" ixy="5.9e-05" iyz="-8.8e-05" ixz="0.000219"/>
-  </inertial>
-  <visual>
-    <origin xyz="0.071615 0.080373 -0.082475" rpy="0 0 0"/>
+    <origin xyz="0.06324664730784718 0.009252948192691707 -0.0658864280055595" rpy="0 0 0"/>
+    <mass value="1.331157749098712"/>
+    <inertia ixx="0.002292" iyy="0.007732" izz="0.008918" ixy="-3.5e-05" iyz="9.1e-05" ixz="0.000807"/>
+  </inertial>
+  <visual>
+    <origin xyz="0.109336 -0.080103 -0.05156" rpy="0 0 0"/>
     <geometry>
       <mesh filename="file://$(find masterHumanoid2025_description)/meshes/left_foot_1.stl" scale="0.001 0.001 0.001"/>
@@ -238,5 +258,5 @@
   </visual>
   <collision>
-    <origin xyz="0.071615 0.080373 -0.082475" rpy="0 0 0"/>
+    <origin xyz="0.109336 -0.080103 -0.05156" rpy="0 0 0"/>
     <geometry>
       <mesh filename="file://$(find masterHumanoid2025_description)/meshes/left_foot_1.stl" scale="0.001 0.001 0.001"/>
@@ -244,95 +264,75 @@
   </collision>
 </link>
-<link name="right_foot_1">
-  <inertial>
-    <origin xyz="0.06874834301237638 0.009252948203182856 -0.060122597886593396" rpy="0 0 0"/>
-    <mass value="1.331157749098713"/>
-    <inertia ixx="0.002203" iyy="0.007732" izz="0.009008" ixy="-4.3e-05" iyz="8.8e-05" ixz="0.000219"/>
-  </inertial>
-  <visual>
-    <origin xyz="0.071369 -0.080103 -0.082473" rpy="0 0 0"/>
-    <geometry>
-      <mesh filename="file://$(find masterHumanoid2025_description)/meshes/right_foot_1.stl" scale="0.001 0.001 0.001"/>
-    </geometry>
-    <material name="silver"/>
-  </visual>
-  <collision>
-    <origin xyz="0.071369 -0.080103 -0.082473" rpy="0 0 0"/>
-    <geometry>
-      <mesh filename="file://$(find masterHumanoid2025_description)/meshes/right_foot_1.stl" scale="0.001 0.001 0.001"/>
-    </geometry>
-  </collision>
-</link>
 <joint name="rotate_12" type="continuous">
-  <origin xyz="-0.009035 0.07965 0.648137" rpy="0 0 0"/>
+  <origin xyz="0.002061 0.07965 0.609638" rpy="0 0 0"/>
   <parent link="base_link"/>
   <child link="left_upper_frame_1"/>
-  <axis xyz="0.0 0.0 -1.0"/>
+  <axis xyz="-0.087156 -0.0 -0.996195"/>
 </joint>
 <joint name="rotate_13" type="continuous">
-  <origin xyz="-0.009035 -0.08035 0.648137" rpy="0 0 0"/>
+  <origin xyz="0.002061 -0.08035 0.609638" rpy="0 0 0"/>
   <parent link="base_link"/>
   <child link="right_upper_frame_1"/>
-  <axis xyz="0.0 0.0 -1.0"/>
+  <axis xyz="-0.087156 -0.0 -0.996195"/>
 </joint>
 <joint name="rotate_10" type="continuous">
-  <origin xyz="-0.06105 6.5e-05 -0.065" rpy="0 0 0"/>
+  <origin xyz="-0.066483 6.5e-05 -0.059432" rpy="0 0 0"/>
   <parent link="left_upper_frame_1"/>
   <child link="left_upper_gearbox_1"/>
-  <axis xyz="-0.999999 0.001062 -0.0"/>
+  <axis xyz="-0.996194 0.001062 0.087156"/>
 </joint>
 <joint name="rotate_11" type="continuous">
-  <origin xyz="-0.06105 0.000111 -0.065" rpy="0 0 0"/>
+  <origin xyz="-0.066483 0.000111 -0.059432" rpy="0 0 0"/>
   <parent link="right_upper_frame_1"/>
   <child link="right_upper_gearbox_1"/>
-  <axis xyz="-0.999998 0.001816 -0.0"/>
+  <axis xyz="-0.996193 0.001816 0.087156"/>
 </joint>
 <joint name="rotate_15" type="continuous">
-  <origin xyz="0.090825 -0.050615 -0.000346" rpy="0 0 0"/>
+  <origin xyz="0.09045 -0.050615 -0.008261" rpy="0 0 0"/>
   <parent link="right_upper_gearbox_1"/>
   <child link="right_middle_leg_1"/>
-  <axis xyz="-0.001816 -0.999998 0.000473"/>
+  <axis xyz="-0.001768 -0.999998 0.000629"/>
 </joint>
 <joint name="rotate_14" type="continuous">
-  <origin xyz="0.09047 0.050354 -0.000321" rpy="0 0 0"/>
+  <origin xyz="0.090099 0.050354 -0.008205" rpy="0 0 0"/>
   <parent link="left_upper_gearbox_1"/>
   <child link="left_middle_leg_1"/>
-  <axis xyz="0.001062 0.999999 0.000972"/>
+  <axis xyz="0.001142 0.999999 0.000876"/>
 </joint>
 <joint name="rotate_16" type="continuous">
-  <origin xyz="-0.000284 0.000243 -0.25" rpy="0 0 0"/>
+  <origin xyz="-0.022072 0.000243 -0.249023" rpy="0 0 0"/>
   <parent link="left_middle_leg_1"/>
   <child link="left_lower_leg_1"/>
-  <axis xyz="0.001062 0.999999 0.000972"/>
+  <axis xyz="0.001142 0.999999 0.000876"/>
 </joint>
 <joint name="rotate_17" type="continuous">
-  <origin xyz="-0.00103 -0.000117 -0.249998" rpy="0 0 0"/>
+  <origin xyz="-0.022815 -0.000117 -0.248957" rpy="0 0 0"/>
   <parent link="right_middle_leg_1"/>
   <child link="right_lower_leg_1"/>
-  <axis xyz="-0.001816 -0.999998 0.000473"/>
+  <axis xyz="-0.001768 -0.999998 0.000629"/>
 </joint>
 <joint name="rotate_19" type="continuous">
-  <origin xyz="0.0 -0.000118 -0.249924" rpy="0 0 0"/>
+  <origin xyz="-0.021782 -0.000118 -0.248972" rpy="0 0 0"/>
   <parent link="right_lower_leg_1"/>
+  <child link="right_lower_gearbox_1"/>
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