Commit message: Update masterHumanoid2025.urdf

File: masterHumanoid2025.urdf (robot description, URDF)
Before this commit: robot masterHumanoid2025, 13 links, 12 joints
Joints:
- joint rotate_19: limit lower=-0.306796 upper=-0.543029 effort=20.0 velocity=5.76 -> lower=0.306796 upper=0.543029 effort=20.0 velocity=5.76
